File: zturn11/zturn11.kicad_pcb (KiCad board)
At the start: 4 copper layers, 266.7 x 215.9 mm, 138 parts, among them J1 2x18edgecon, J11 Conn_02x40_Odd_Even, J12 Conn_02x40_Odd_Even, J2 2x18edgecon, J3 2x18edgecon, J4 2x18edgecon, J5 Conn_01x16, J7 Conn_01x03, Q1 SSM6N15AFU, Q10 SSM6N15AFU, Q11 SSM6N15AFU, Q12 SSM6N15AFU, Q13 SSM6N15AFU, Q14 SSM6N15AFU, Q15 SSM6N15AFU, Q16 SSM6N15AFU, Q17 SSM6N15AFU, Q18 SSM6N15AFU, Q19 SSM6N15AFU, Q2 SSM6N15AFU, Q20 SSM6N15AFU, Q21 SSM6N15AFU, Q22 SSM6N15AFU, Q23 SSM6N15AFU, Q24 SSM6N15AFU, Q25 SSM6N15AFU, Q26 SSM6N15AFU, Q27 SSM6N15AFU, Q28 SSM6N15AFU, Q29 SSM6N15AFU, Q3 SSM6N15AFU, Q30 SSM6N15AFU, Q31 SSM6N15AFU, Q32 SSM6N15AFU, Q33 SSM6N15AFU, Q34 SSM6N15AFU, Q35 SSM6N15AFU, Q36 SSM6N15AFU, Q37 SSM6N15AFU, Q38 SSM6N15AFU, Q39 SSM6N15AFU, Q4 SSM6N15AFU, Q40 SSM6N15AFU, Q41 SSM6N15AFU, Q42 SSM6N15AFU, Q43 SSM6N15AFU, Q44 SSM6N15AFU, Q5 SSM6N15AFU, Q50 SSM6N15AFU, Q51 SSM6N15AFU, Q52 SSM6N15AFU, Q53 SSM6N15AFU, Q54 SSM6N15AFU, Q55 SSM6N15AFU, Q56 SSM6N15AFU, Q57 SSM6N15AFU, Q58 SSM6N15AFU, Q59 SSM6N15AFU, Q6 SSM6N15AFU, Q60 SSM6N15AFU, Q61 SSM6N15AFU, Q62 SSM6N15AFU, Q63 SSM6N15AFU, Q64 SSM6N15AFU, Q7 SSM6N15AFU, Q8 SSM6N15AFU, Q9 SSM6N15AFU

Commit message: update pcb with patch for BG6_OUT_H
also move power connector out from under zturn board
Parts:
- moved J7 35.9 mm to (61.0, 127.0)
Connections:
- J11 pad 45: /BR6_OUT_H -> unconnected-(J11-Pin_45-Pad45)
- J12 pad 57: /IOB35LP15 -> /BR6_OUT_H
- J5 pad 14: /IOB35LP15 -> unconnected-(J5-Pin_14-Pad14)
Routing:
- net /V5ZYNQ: track 85.9 -> 139.4 mm
- net /BR6_OUT_H: track 113.6 -> 141.8 mm, vias 0 -> 3
- net /IOB35LP15: track 13.4 -> 0.00 mm
- net /D14_OUT_H: track 175.3 -> 177.4 mm
- net /D15_OUT_H: track 180.3 -> 182.4 mm
- net /D13_OUT_H: track 170.3 -> 172.3 mm
- net /D09_OUT_H: track 154.0 -> 156.0 mm
- net /D12_OUT_H: track 165.3 -> 167.3 mm
- net /D10_OUT_H: track 159.0 -> 161.0 mm
- net /D08_OUT_H: track 149.0 -> 151.0 mm
- net /NPG_OUT_L: track 172.3 -> 171.3 mm
Other:
- board text added: "ZTURN11-2024-04-24"
- board text removed: "ZTURN11-2024-04-13"

Commit message: add diodes to the zturn11 board so the muxes work
also add AC_LO_OUT_H and DC_LO_OUT_H drivers
Parts:
- added C20: 0.1u, Capacitor_SMD:C_0402_1005Metric, F.Cu at (149.2, 69.8)
- added D1: RB521S-30, Diode_SMD:D_SOD-523, F.Cu at (248.0, 181.6)
- added D10: RB521S-30, Diode_SMD:D_SOD-523, F.Cu at (91.8, 181.6)
- added D11: RB521S-30, Diode_SMD:D_SOD-523, F.Cu at (86.0, 181.6)
- added D12: RB521S-30, Diode_SMD:D_SOD-523, F.Cu at (80.3, 181.6)
- added D13: RB521S-30, Diode_SMD:D_SOD-523, F.Cu at (74.6, 181.6)
- added D14: RB521S-30, Diode_SMD:D_SOD-523, F.Cu at (68.9, 181.6)
- added D15: RB521S-30, Diode_SMD:D_SOD-523, F.Cu at (35.2, 181.6)
- added D16: RB521S-30, Diode_SMD:D_SOD-523, B.Cu at (230.8, 181.6)
- added D17: RB521S-30, Diode_SMD:D_SOD-523, B.Cu at (235.3, 181.6)
- added D18: RB521S-30, Diode_SMD:D_SOD-523, B.Cu at (239.7, 181.6)
- added D19: RB521S-30, Diode_SMD:D_SOD-523, B.Cu at (244.2, 181.6)
- added D2: RB521S-30, Diode_SMD:D_SOD-523, F.Cu at (237.5, 181.6)
- added D20: RB521S-30, Diode_SMD:D_SOD-523, B.Cu at (248.6, 181.6)
- added D21: RB521S-30, Diode_SMD:D_SOD-523, B.Cu at (253.0, 181.6)
- added D22: RB521S-30, Diode_SMD:D_SOD-523, B.Cu at (257.5, 181.6)
- added D23: RB521S-30, Diode_SMD:D_SOD-523, B.Cu at (261.9, 181.6)
- added D24: RB521S-30, Diode_SMD:D_SOD-523, B.Cu at (226.4, 181.6)
- added D25: RB521S-30, Diode_SMD:D_SOD-523, B.Cu at (221.9, 181.6)
- added D26: RB521S-30, Diode_SMD:D_SOD-523, B.Cu at (217.5, 181.6)
- added D27: RB521S-30, Diode_SMD:D_SOD-523, B.Cu at (213.0, 181.6)
- added D28: RB521S-30, Diode_SMD:D_SOD-523, B.Cu at (208.6, 181.6)
- added D29: RB521S-30, Diode_SMD:D_SOD-523, B.Cu at (204.2, 181.6)
- added D3: RB521S-30, Diode_SMD:D_SOD-523, F.Cu at (223.8, 181.6)
- added D30: RB521S-30, Diode_SMD:D_SOD-523, B.Cu at (199.7, 181.6)
- added D31: RB521S-30, Diode_SMD:D_SOD-523, B.Cu at (188.3, 181.6)
- added D32: RB521S-30, Diode_SMD:D_SOD-523, B.Cu at (117.2, 182.2)
- added D33: RB521S-30, Diode_SMD:D_SOD-523, B.Cu at (122.9, 181.6)
- added D34: RB521S-30, Diode_SMD:D_SOD-523, B.Cu at (128.6, 181.6)
- added D35: RB521S-30, Diode_SMD:D_SOD-523, B.Cu at (111.4, 181.6)
- added D36: RB521S-30, Diode_SMD:D_SOD-523, B.Cu at (105.7, 181.6)
- added D37: RB521S-30, Diode_SMD:D_SOD-523, B.Cu at (100.0, 181.6)
- added D38: RB521S-30, Diode_SMD:D_SOD-523, B.Cu at (94.3, 181.6)
- added D39: RB521S-30, Diode_SMD:D_SOD-523, B.Cu at (88.6, 181.6)
- added D4: RB521S-30, Diode_SMD:D_SOD-523, F.Cu at (207.3, 181.6)
- added D40: RB521S-30, Diode_SMD:D_SOD-523, B.Cu at (82.9, 181.6)
- added D41: RB521S-30, Diode_SMD:D_SOD-523, B.Cu at (77.2, 181.6)
- added D42: RB521S-30, Diode_SMD:D_SOD-523, B.Cu at (182.6, 181.6)
- added D43: RB521S-30, Diode_SMD:D_SOD-523, B.Cu at (176.8, 181.6)
- added D44: RB521S-30, Diode_SMD:D_SOD-523, B.Cu at (171.1, 181.6)
- added D5: RB521S-30, Diode_SMD:D_SOD-523, F.Cu at (131.8, 181.6)
- added D6: RB521S-30, Diode_SMD:D_SOD-523, F.Cu at (126.0, 181.6)
- added D7: RB521S-30, Diode_SMD:D_SOD-523, F.Cu at (114.6, 181.6)
- added D8: RB521S-30, Diode_SMD:D_SOD-523, F.Cu at (108.9, 181.6)
- added D9: RB521S-30, Diode_SMD:D_SOD-523, F.Cu at (97.8, 181.6)
- C8: moved to B.Cu
- moved R1 15.7 mm to (146.2, 69.8), turned to 180 degrees
- moved R6 2.54 mm to (153.0, 76.8)
- moved R4 1.27 mm to (155.6, 76.8)
Connections:
- J11 pad 41: /D06_OUT_H -> /BR7_OUT_H
- J11 pad 43: /BR7_OUT_H -> /BR6_OUT_H
- J12 pad 46: /PB_OUT_H -> /AC_LO_OUT_H
- J12 pad 48: /RSEL1_H -> /PB_OUT_H
- J12 pad 52: /D02_OUT_H -> /D06_OUT_H
- J12 pad 53: /IOB35LP13 -> /NPG_OUT_L
- J12 pad 54: /D03_OUT_H -> /D02_OUT_H
- J12 pad 55: /IOB35LN13 -> /D15_OUT_H
- J12 pad 56: /D00_OUT_H -> /D03_OUT_H
- J12 pad 57: /BR6_OUT_H -> /NPG_IN_L
- J12 pad 58: /D01_OUT_H -> /D00_OUT_H
- J12 pad 59: /NPG_OUT_L -> /D14_OUT_H
- J12 pad 62: /D05_OUT_H -> /D01_OUT_H
- J12 pad 63: /D15_OUT_H -> /PA_OUT_H
- J12 pad 64: /D04_OUT_H -> /D05_OUT_H
- J12 pad 65: /D14_OUT_H -> /D13_OUT_H
- J12 pad 66: /D07_OUT_H -> /D04_OUT_H
- J12 pad 67: /D13_OUT_H -> /D12_OUT_H
- J12 pad 68: /HLTGR_IN_L -> /RSEL1_H
- J12 pad 69: /D12_OUT_H -> /D10_OUT_H
- J12 pad 72: /HLTRQ_OUT_H -> /HLTGR_IN_L
- J12 pad 73: /D10_OUT_H -> /D09_OUT_H
- J12 pad 74: /DC_LO_IN_H -> /HLTRQ_OUT_H
- J12 pad 75: /D09_OUT_H -> /D08_OUT_H
- J12 pad 76: /D11_OUT_H -> /DC_LO_IN_H
- J12 pad 77: /D08_OUT_H -> /D07_OUT_H
- J12 pad 78: /PA_OUT_H -> /DC_LO_OUT_H
- J12 pad 79: /NPG_IN_L -> /D11_OUT_H
- J5 pad 12: /IOB35LP13 -> unconnected-(J5-Pin_12-Pad12)
- J5 pad 13: /IOB35LN13 -> unconnected-(J5-Pin_13-Pad13)
- J5 pad 4: unconnected-(J5-Pin_4-Pad4) -> +3V3
- Q10 pad 6: /MUXA -> Net-(D5-K)
- Q11 pad 6: /MUXB -> Net-(D6-K)
- Q13 pad 6: /MUXC -> Net-(D7-K)
- Q14 pad 6: /MUXA -> Net-(D8-K)
- Q16 pad 6: /MUXB -> Net-(D9-K)
- Q17 pad 6: /MUXC -> Net-(D10-K)
- Q18 pad 6: /MUXD -> Net-(D11-K)
- Q19 pad 6: /MUXE -> Net-(D12-K)
- Q2 pad 6: /MUXA -> Net-(D1-K)
- Q20 pad 6: /MUXF -> Net-(D13-K)
- Q21 pad 6: /MUXH -> Net-(D14-K)
- Q23 pad 6: /MUXJ -> Net-(D15-K)
- Q25 pad 6: /MUXE -> Net-(D23-K)
- Q26 pad 6: /MUXF -> Net-(D22-K)
- Q27 pad 6: /MUXH -> Net-(D21-K)
- Q28 pad 6: /MUXJ -> Net-(D20-K)
- Q29 pad 6: /MUXK -> Net-(D19-K)
- Q3 pad 6: /MUXB -> Net-(D2-K)
- Q30 pad 6: /MUXL -> Net-(D18-K)
- Q31 pad 6: /MUXM -> Net-(D17-K)
- Q32 pad 6: /MUXN -> Net-(D16-K)
- Q33 pad 6: /MUXP -> Net-(D24-K)
- Q34 pad 6: /MUXR -> Net-(D25-K)
- Q35 pad 6: /MUXS -> Net-(D26-K)
- Q36 pad 6: /MUXD -> Net-(D27-K)
- Q37 pad 6: /MUXE -> Net-(D28-K)
- Q38 pad 6: /MUXF -> Net-(D29-K)
- Q39 pad 6: /MUXH -> Net-(D30-K)
- Q4 pad 3: unconnected-(Q4B-D2-Pad3) -> /BUS_DC_LO_L
- Q4 pad 5: unconnected-(Q4B-G2-Pad5) -> /DC_LO_OUT_H
- Q40 pad 6: /MUXJ -> Net-(D31-K)
- Q41 pad 6: /MUXK -> Net-(D42-K)
- Q42 pad 6: /MUXL -> Net-(D43-K)
- Q43 pad 6: /MUXM -> Net-(D44-K)
- Q5 pad 6: /MUXC -> Net-(D3-K)
- Q54 pad 6: /MUXN -> Net-(D34-K)
- Q55 pad 6: /MUXP -> Net-(D33-K)
- Q56 pad 6: /MUXR -> Net-(D32-K)
- Q57 pad 6: /MUXK -> Net-(D35-K)
- Q58 pad 6: /MUXL -> Net-(D36-K)
- Q59 pad 6: /MUXM -> Net-(D37-K)
- Q60 pad 6: /MUXN -> Net-(D38-K)
- Q61 pad 6: /MUXP -> Net-(D39-K)
- Q62 pad 6: /MUXR -> Net-(D40-K)
- Q63 pad 6: /MUXS -> Net-(D41-K)
- Q7 pad 6: /MUXD -> Net-(D4-K)
- Q8 pad 3: unconnected-(Q8B-D2-Pad3) -> /BUS_AC_LO_L
- Q8 pad 5: unconnected-(Q8B-G2-Pad5) -> /AC_LO_OUT_H
Routing:
- net /DC_LO_OUT_H: track 0.00 -> 142.7 mm
- net /AC_LO_OUT_H: track 0.00 -> 141.7 mm
- net /BR6_OUT_H: track 141.8 -> 114.8 mm, vias 3 -> 0
- net /NPG_IN_L: track 155.6 -> 176.1 mm
- net /MUXA: track 293.7 -> 274.2 mm
- net /MUXD: track 256.7 -> 238.4 mm
- net /MUXB: track 278.0 -> 260.8 mm, vias 5 -> 4
- net /MUXC: track 264.8 -> 247.8 mm
- net /MUXM: track 287.7 -> 271.5 mm
- net /MUXL: track 295.0 -> 278.9 mm
- net /MUXN: track 277.1 -> 261.3 mm
- net /MUXF: track 306.1 -> 290.3 mm
- net /MUXK: track 301.6 -> 285.9 mm
- net /MUXE: track 313.1 -> 297.3 mm
- net /MUXP: track 272.3 -> 256.6 mm
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Other:
- board text added: "ZTURN11-2024-04-28"
- board text removed: "ZTURN11-2024-04-24"
